Commit message: Putting Xarm6 in the my_moveit_resources

File: src/my_moveit_resources/xarm6/xarm6_moveit_config/config/xarm6.ros2_control.xacro (robot description, xacro)
@@ -1,16 +1,10 @@
 <?xml version="1.0"?>
 <robot xmlns:xacro="http://www.ros.org/wiki/xacro">
-    <xacro:macro name="xarm6_ros2_control" params="name initial_positions_file ros2_control_hardware_type">
-        <xacro:property name="initial_positions" value="${xacro.load_yaml(initial_positions_file)['initial_positions']}"/>
+    <xacro:macro name="xarm6_ros2_control" params="name initial_positions_file">
+        <xacro:property name="initial_positions" value="${load_yaml(initial_positions_file)['initial_positions']}"/>
         <ros2_control name="${name}" type="system">
             <hardware>
-                <xacro:if value="${ros2_control_hardware_type == 'mock_components'}">
-                    <plugin>mock_components/GenericSystem</plugin>
-                </xacro:if>
-                <xacro:if value="${ros2_control_hardware_type == 'isaac'}">
-                    <plugin>topic_based_ros2_control/TopicBasedSystem</plugin>
-                    <param name="joint_commands_topic">/isaac_joint_commands</param>
-                    <param name="joint_states_topic">/isaac_joint_states</param>
-                </xacro:if>
+                <!-- By default, set up controllers for simulation. This won't work on real hardware -->
+                <plugin>mock_components/GenericSystem</plugin>
             </hardware>
             <joint name="joint1">

File: src/my_moveit_resources/xarm6/xarm6_moveit_config/config/xarm6.urdf.xacro (robot description, xacro)
@@ -1,12 +1,9 @@
 <?xml version="1.0"?>
-<robot xmlns:xacro="http://ros.org/wiki/xacro" name="xarm6">
+<robot xmlns:xacro="http://www.ros.org/wiki/xacro" name="xarm6">
     <xacro:arg name="initial_positions_file" default="initial_positions.yaml" />
-    <xacro:arg name="ros2_control_hardware_type" default="mock_components" />
     <!-- Import xarm6 urdf file -->
-    <xacro:include filename="$(find my_moveit_xarm6_description)/urdf/xarm6_without_gripper.urdf" />
-    <!-- Import xarm6 ros2_control description -->
+    <xacro:include filename="$(find my_moveit_xarm6_description)/urdf/xarm6.urdf" />
+    <!-- Import control_xacro -->
     <xacro:include filename="xarm6.ros2_control.xacro" />
-    <xacro:include filename="xarm6_gripper.ros2_control.xacro" />
-    <xacro:xarm6_ros2_control name="Xarm6FakeSystem" initial_positions_file="$(arg initial_positions_file)" ros2_control_hardware_type="$(arg ros2_control_hardware_type)"/>
-    <xacro:xarm6_gripper_ros2_control name="Xarm6HandFakeSystem" ros2_control_hardware_type="$(arg ros2_control_hardware_type)"/>
+    <xacro:xarm6_ros2_control name="FakeSystem" initial_positions_file="$(arg initial_positions_file)"/>
 </robot>
